File: Ročníkový projekt S3E.kicad_pcb (KiCad board)
At the start: 2 copper layers, 36 parts, among them IC1 PIC18F47Q43-I_P, IC3 ULN2804A, IC5 MCP7940M-I_SN, J1 DG126-5.0-02P-14-00A, J2 - nastavení času, J3 + nastavení času, J4 826632-9, J5 826632-9, J6 826632-9, J7 TSW-105-07-G-S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

Commit message: backup update
Parts:
- removed J4, J5, J6: 826632-9, SamacSys_Parts:HDRV18W85P254_2X9_2286X500X970P
- added C6: 100nF, Capacitor_SMD:C_1206_3216Metric_Pad1.33x1.80mm_HandSolder, B.Cu at (170.9, 58.1)
- added R13: 4.7k, Resistor_SMD:R_1206_3216Metric_Pad1.30x1.75mm_HandSolder, B.Cu at (159.4, 59.9)
- added R14: 470R, Resistor_SMD:R_1206_3216Metric_Pad1.30x1.75mm_HandSolder, B.Cu at (160.9, 63.6)
- added S1: S, My parts:Screen_connector_footprint_parraler, F.Cu at (244.3, 97.2)
- IC5: footprint My parts:SOIC127P600X175-8N -> SamacSys_Parts:SOIC127P600X175-8N
- moved Q1 110.5 mm to (154.7, 110.5)
- moved Q5 104.9 mm to (154.6, 90.1)
- moved Q6 98.5 mm to (154.7, 95.4)
- moved Q3 92.6 mm to (154.5, 100.2)
- moved Q4 86.1 mm to (154.5, 105.3)
- moved Q2 73.7 mm to (185.4, 115.8), turned to 90 degrees
- moved J1 59.7 mm to (174.3, 45.4), turned to 180 degrees
- moved R4 34.8 mm to (170.9, 65.4), turned to 0 degrees
- moved R3 30.9 mm to (170.9, 68.4), turned to 0 degrees
- moved R19 27.1 mm to (170.9, 71.2), turned to 0 degrees
- moved C3 27.1 mm to (165.6, 117.4)
- moved J7 21.3 mm to (168.4, 53.4)
- moved IC3 20.2 mm to (192.2, 96.5)
- moved R5 19.6 mm to (203.3, 80.2)
- moved IC1 19.6 mm to (173.8, 87.7)
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Connections:
- IC1 pad 1: MCLR -> Net-(IC1-~{MCLR}/VPP/RE3)
- IC1 pad 13: unconnected-(IC1-RA7-Pad13) -> A_6
- IC1 pad 14: A_6 -> A_5
- IC1 pad 15: A_5 -> A_4
- IC1 pad 16: A_4 -> A_3
- IC1 pad 17: A_3 -> A_2
- IC1 pad 19: A_2 -> unconnected-(IC1-RD0-Pad19)
- IC1 pad 20: A_1 -> unconnected-(IC1-RD1-Pad20)
- IC1 pad 21: unconnected-(IC1-RD2-Pad21) -> A_1
- IC1 pad 22: unconnected-(IC1-RD3-Pad22) -> PIC_G
- IC1 pad 24: PIC_G -> PIC_F
- IC1 pad 25: PIC_F -> PIC_E
- IC1 pad 26: PIC_E -> PIC_D
- IC1 pad 27: PIC_D -> PIC_C
- IC1 pad 28: PIC_C -> PIC_B
- IC1 pad 29: PIC_B -> PIC_A
- IC1 pad 30: PIC_A -> PIC_DP
- IC1 pad 33: PIC_DP -> unconnected-(IC1-RB0-Pad33)
- J7 pad 1: MCLR -> Net-(J7-Pad1)
- Q1 pad 2: A_6 -> A_2
- Q2 pad 2: A_5 -> A_1
- Q5 pad 2: A_2 -> A_6
- Q6 pad 2: A_1 -> A_5
Routing:
- net VDD_P: track 239.0 -> 149.1 mm, vias 0 -> 1
- net Net-(Q2-C): track 0.00 -> 44.7 mm
- net Net-(IC1-RA0): track 36.9 -> 12.3 mm
- net Net-(IC1-RA1): track 32.2 -> 13.9 mm
- net Net-(C6-Pad1): track 0.00 -> 13.5 mm
- net A_2: track 0.00 -> 12.6 mm
- net A_6: track 0.00 -> 12.6 mm
- net A_3: track 0.00 -> 11.6 mm
- net A_5: track 0.00 -> 11.5 mm
- net Net-(J7-Pad1): track 0.00 -> 11.0 mm
- net /DP': track 21.6 -> 32.4 mm
- net /G': track 20.8 -> 31.5 mm
- net /F': track 20.0 -> 30.6 mm
- net A_4: track 0.00 -> 10.6 mm
- net /D': track 21.1 -> 30.9 mm
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- added copper zone on B.Cu, net VDD_P
Other:
- board outline added: 99 x 92 mm

Commit message: backup update
Parts:
- moved Q1 46.5 mm to (187.7, 77.7), turned to 180 degrees
- moved S1 46.1 mm to (204.0, 74.8), turned to 90 degrees
- moved Q4 46.0 mm to (187.7, 73.4), turned to 180 degrees
- moved Q3 45.6 mm to (187.7, 69.0), turned to 180 degrees
- moved Q6 45.3 mm to (187.8, 64.4), turned to 180 degrees
- moved Q5 44.6 mm to (187.7, 60.1), turned to 180 degrees
- moved Q2 33.7 mm to (187.7, 82.2), turned to 180 degrees
- moved R10 5.95 mm to (197.4, 105.0)
- moved R11 5.95 mm to (197.4, 109.7)
- moved R12 5.95 mm to (197.4, 114.5)
- moved R5 5.95 mm to (197.4, 81.2)
- moved R6 5.95 mm to (197.4, 86.0)
- moved R7 5.95 mm to (197.4, 90.7)
- moved R8 5.95 mm to (197.4, 95.5)
- moved R9 5.95 mm to (197.4, 100.2)
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Connections:
- IC1 pad 13: A_6 -> unconnected-(IC1-RA7-Pad13)
- IC1 pad 14: A_5 -> unconnected-(IC1-RA6-Pad14)
- IC1 pad 15: A_4 -> unconnected-(IC1-RC0-Pad15)
- IC1 pad 16: A_3 -> unconnected-(IC1-RC1-Pad16)
- IC1 pad 17: A_2 -> unconnected-(IC1-RC2-Pad17)
- IC1 pad 21: A_1 -> unconnected-(IC1-RD2-Pad21)
- IC1 pad 33: unconnected-(IC1-RB0-Pad33) -> A_1
- IC1 pad 34: unconnected-(IC1-RB1-Pad34) -> A_2
- IC1 pad 35: unconnected-(IC1-RB2-Pad35) -> A_3
- IC1 pad 36: unconnected-(IC1-RB3-Pad36) -> A_4
- IC1 pad 37: unconnected-(IC1-RB4-Pad37) -> A_5
- IC1 pad 38: unconnected-(IC1-RB5-Pad38) -> A_6
- S1 pad 1: Net-(Q5-C) -> Net-(Q2-C)
- S1 pad 10: Net-(Q3-C) -> Net-(Q4-C)
- S1 pad 19: Net-(Q1-C) -> Net-(Q6-C)
- S1 pad 36: Net-(Q2-C) -> Net-(Q5-C)
- S1 pad 45: Net-(Q4-C) -> Net-(Q3-C)
- S1 pad 54: Net-(Q6-C) -> Net-(Q1-C)
Routing:
- net VDD_P: track 149.1 -> 97.0 mm, vias 1 -> 0
- net Net-(Q2-C): track 44.7 -> 9.41 mm
- net /A': track 35.2 -> 66.9 mm
- net /B': track 33.0 -> 61.1 mm
- net /C': track 31.8 -> 55.3 mm
- net /D': track 30.9 -> 49.5 mm
- net /E': track 30.0 -> 44.5 mm
- net Net-(Q6-C): track 0.00 -> 12.3 mm
- net Net-(Q4-C): track 0.00 -> 11.0 mm
- net Net-(Q5-C): track 0.00 -> 10.6 mm
- net /F': track 30.6 -> 39.8 mm
- net Net-(Q3-C): track 0.00 -> 9.14 mm
- net Net-(Q1-C): track 0.00 -> 7.82 mm
- net A_2: track 12.6 -> 5.28 mm
- net A_3: track 11.6 -> 5.96 mm
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Other:
- board size 99 x 92 mm -> 64 x 92 mm

Commit message: backup update
Parts:
- moved C4 0.50 mm to (177.9, 85.2)
Routing:
- net VDD_P: track 97.0 -> 121.5 mm, vias 0 -> 2
Changed lines of the file:
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@@
 	(footprint "Capacitor_SMD:C_1206_3216Metric_Pad1.33x1.80mm_HandSolder"
 		(layer "B.Cu")
-		(at 178.4 85.1375 90)
+		(at 177.9 85.1625 90)
 		(descr "Capacitor SMD 1206 (3216 Metric), square (rectangular) end terminal, IPC-7351 nominal with elongated pad for handsoldering. (Body size source: IPC-SM-782 page 76, https://www.pcb-3d.com/wordpress/wp-content/uploads/ipc-sm-782a_amendment_1_and_2.pdf), generated with kicad-footprint-generator")
 		(tags "capacitor handsolder")
@@
 	)
 	(segment
+		(start 176 89.3)
+		(end 176 71.312595)
+		(width 0.5)
+		(layer "F.Cu")
+		(net 60)
+	)
+	(segment
+		(start 176 71.312595)
+		(end 176.038884 71.273711)
+		(width 0.5)
+		(layer "F.Cu")
+		(net 60)
+	)
+	(via
+		(at 176.038884 71.273711)
+		(size 0.6)
+		(drill 0.3)
+		(layers "F.Cu" "B.Cu")
+		(net 60)
+	)
+	(via
+		(at 176 89.3)
+		(size 0.6)
+		(drill 0.3)
+		(layers "F.Cu" "B.Cu")
+		(net 60)
+	)
+	(segment
 		(start 180.7 123.1)
 		(end 184.9 118.9)
@@
 	)
 	(segment
+		(start 175.965173 71.2)
+		(end 176.038884 71.273711)
+		(width 0.5)
+		(layer "B.Cu")
+		(net 60)
+	)
+	(segment
 		(start 172.5 58.1)
 		(end 172.5 71.2)
@@
 	)
 	(segment
-		(start 171.15 86.4)
+		(start 172.5 71.2)
+		(end 175.965173 71.2)
+		(width 0.5)
+		(layer "B.Cu")
+		(net 60)
+	)
+	(segment
+		(start 176 86.4)
 		(end 181.5 86.4)
 		(width 0.7)
@@
 	)
 	(segment
+		(start 171.15 86.4)
+		(end 176 86.4)
+		(width 0.7)
+		(layer "B.Cu")
+		(net 60)
+	)
+	(segment
 		(start 184.9 109.28)
 		(end 187.2 109.28)
@@
 		(width 0.5)
 		(layer "B.Cu")
+		(net 60)
+	)
+	(segment
+		(start 176 86.4)
+		(end 176 89.3)
+		(width 0.5)
+		(layer "B.Cu")

Commit message: backup update
Parts:
- added C7: 100uF, Capacitor_THT:CP_Radial_D6.3mm_P2.50mm, F.Cu at (183.7, 46.7)
- added C8: 100uF, Capacitor_THT:CP_Radial_D6.3mm_P2.50mm, F.Cu at (194.4, 46.7)
- C1, C2: footprint Capacitor_SMD:C_0603_1608Metric_Pad1.08x0.95mm_HandSolder -> Capacitor_SMD:C_0805_2012Metric_Pad1.18x1.45mm_HandSolder
Routing:
- net VCC_P: track 171.9 -> 199.6 mm
- net VDD_P: track 121.5 -> 142.0 mm

Commit message: backup update
Parts:
- added D1: M7 SMD T/R, Diode_SMD:D_SMA_Handsoldering, B.Cu at (198.4, 47.8)
- moved J1 38.8 mm to (213.1, 44.6)
- moved C7 4.98 mm to (178.8, 45.8)
- moved C8 4.89 mm to (189.6, 45.8)
Connections:
- J1 pad 1: VDD_P -> Net-(D1-K)
Routing:
- net Net-(D1-K): track 0.00 -> 13.5 mm
- net VCC_P: track 199.6 -> 207.1 mm
- net VDD_P: track 142.0 -> 141.0 mm
Other:
- board text added: "+ -"
- board text added: "DAT CLK GND VCC MCLR"
