File: Ročníkový projekt S3E.kicad_pcb (KiCad board)
At the start: 2 copper layers, 64 x 92 mm, 40 parts, among them IC1 PIC18F47Q43-I_P, IC3 ULN2804A, IC5 MCP7940M-I_SN, J1 DG126-5.0-02P-14-00A, J2 - nastavení času, J3 + nastavení času, J7 TSW-105-07-G-S, J8 přepínání mezi číslicemi, Q1 DTA123JCAT116, Q2 DTA123JCAT116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

Commit message: backup update
Parts:
- moved S1 0.31 mm to (204.3, 74.6)
Connections:
- S1 pad 19: Net-(Q6-C) -> Net-(Q5-C)
- S1 pad 20: /A' -> Net-(Q6-C)
- S1 pad 21: /B' -> /A'
- S1 pad 22: /C' -> /B'
- S1 pad 23: /D' -> /C'
- S1 pad 24: /E' -> /D'
- S1 pad 25: /F' -> /E'
- S1 pad 26: /G' -> /F'
- S1 pad 27: /DP' -> /G'
- S1 pad 29: /G' -> /DP'
- S1 pad 30: /F' -> /G'
- S1 pad 31: /E' -> /F'
- S1 pad 32: /D' -> /E'
- S1 pad 33: /C' -> /D'
- S1 pad 34: /B' -> /C'
- S1 pad 35: /A' -> /B'
- S1 pad 36: Net-(Q5-C) -> /A'
- S1 pad 37: /DP' -> Net-(Q3-C)
- S1 pad 38: /G' -> /DP'
- S1 pad 39: /F' -> /G'
- S1 pad 40: /E' -> /F'
- S1 pad 41: /D' -> /E'
- S1 pad 42: /C' -> /D'
- S1 pad 43: /B' -> /C'
- S1 pad 44: /A' -> /B'
- S1 pad 45: Net-(Q3-C) -> /A'
- S1 pad 46: /DP' -> Net-(Q1-C)
Routing:
- net Net-(Q6-C): track 12.3 -> 14.7 mm
- net Net-(Q5-C): track 10.6 -> 9.35 mm

Commit message: backup update
Parts:
- IC5: footprint SamacSys_Parts:SOIC127P600X175-8N -> My parts:SOIC127P600X175-8N
Changed lines of the file:
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@@
 		)
 	)
-	(footprint "SamacSys_Parts:SOIC127P600X175-8N"
+	(footprint "My parts:SOIC127P600X175-8N"
 		(layer "B.Cu")
 		(at 173.4 117.7)
-		(descr "8-LEAD PLASTIC SMALL OUTLINE (SN)-ren1")
+		(descr "MCP7940M-I/SN")
 		(tags "Integrated Circuit")
 		(property "Reference" "IC5"
@@
 		)
 		(embedded_fonts no)
-		(model "/home/nontoxiccat/Kicad Libs/SamacSys/SamacSys_Parts.3dshapes/MCP7940N-I_SN.stp"
+		(model "${KICAD9_3RD_PARTY}/MCP7940M-I_SN.stp"
 			(offset
 				(xyz 0 0 0)

Commit message: backup update
Parts:
- added C10: 100nF, Capacitor_SMD:C_1206_3216Metric_Pad1.33x1.80mm_HandSolder, B.Cu at (162.3, 41.9)
- added C9: 100nF, Capacitor_SMD:C_1206_3216Metric_Pad1.33x1.80mm_HandSolder, B.Cu at (166.6, 49.9)
- added IC2: L7805CD2T-TR, My parts:L7805CD2T, B.Cu at (171.7, 42.9)
- moved C7 18.5 mm to (196.1, 39.1), turned to -90 degrees
- moved D1 12.7 mm to (210.8, 45.4)
- moved J1 7.23 mm to (208.3, 39.1), turned to 0 degrees
- moved C8 6.67 mm to (188.5, 39.2), turned to -90 degrees
- moved J7 1.96 mm to (168.4, 55.4)
- moved C6 1.35 mm to (171.0, 59.5)
Connections:
- C7 pad 1: VDD_P -> Net-(IC2-INPUT)
- C7 pad 2: VCC_P -> VDD_P
- C8 pad 1: VDD_P -> Net-(IC2-INPUT)
- C8 pad 2: VCC_P -> VDD_P
- J1 pad 1: Net-(D1-K) -> Net-(IC2-INPUT)
- J1 pad 2: VCC_P -> Net-(D1-K)
Routing:
- net Net-(IC2-INPUT): track 0.00 -> 51.0 mm, vias 0 -> 2
- net VDD_P: track 141.0 -> 179.8 mm, vias 2 -> 4
- net VCC_P: track 207.1 -> 182.3 mm
- net Net-(D1-K): track 13.5 -> 6.20 mm
- net ICSP_DAT: track 11.4 -> 9.41 mm
- net ICSP_CLK: track 15.0 -> 13.0 mm
- net Net-(J7-Pad1): track 11.0 -> 10.2 mm
- net Net-(C6-Pad1): track 13.5 -> 13.0 mm
Other:
- board size 64 x 92 mm -> 64 x 95.3 mm
