File: Ročníkový projekt S3E.kicad_sch (KiCad schematic)
At the start: 36 parts, among them IC1 PIC18F47Q43-I_P, IC3 ULN2804A, IC5 MCP7940M-I_SN, J1 DG126-5.0-02P-14-00A, J2 - nastavení času, J3 + nastavení času, J4 826632-9, J5 826632-9, J6 826632-9, J7 TSW-105-07-G-S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

Commit message: backup update
Parts:
- removed J4, J5, J6: 826632-9, SamacSys_Parts:HDRV18W85P254_2X9_2286X500X970P, symbol SamacSys_Parts:826632-9
- added C6: 100nF, Capacitor_SMD:C_1206_3216Metric_Pad1.33x1.80mm_HandSolder, symbol Device:C_Small
- added R13: 4.7k, Resistor_SMD:R_1206_3216Metric_Pad1.30x1.75mm_HandSolder, symbol Device:R_Small
- added R14: 470R, Resistor_SMD:R_1206_3216Metric_Pad1.30x1.75mm_HandSolder, symbol Device:R_Small
- added S1: S, My parts:Screen_connector_footprint_parraler, symbol My_parts:Screen_connector_symbol
- IC5: footprint SOIC127P600X175-8N -> SamacSys_Parts:SOIC127P600X175-8N
Connections:
- net A': now also S1.11, S1.2, S1.20, S1.35, S1.44, S1.53
- net A_1: now also IC1.21 (RD2), Q2.2 (B); no longer IC1.20 (RD1), Q6.2 (B)
- net A_2: now also IC1.17 (RC2), Q1.2 (B); no longer IC1.19 (RD0), Q5.2 (B)
- net A_3: now also IC1.16 (RC1); no longer IC1.17 (RC2)
- net A_4: now also IC1.15 (RC0); no longer IC1.16 (RC1)
- net A_5: now also IC1.14 (RA6), Q6.2 (B); no longer IC1.15 (RC0), Q2.2 (B)
- net A_6: now also IC1.13 (RA7), Q5.2 (B); no longer IC1.14 (RA6), Q1.2 (B)
- net B': now also S1.12, S1.21, S1.3, S1.34, S1.43, S1.52
- net C': now also S1.13, S1.22, S1.33, S1.4, S1.42, S1.51
- net D': now also S1.14, S1.23, S1.32, S1.41, S1.5, S1.50
- net DP': now also S1.18, S1.27, S1.28, S1.37, S1.46, S1.9
- net E': now also S1.15, S1.24, S1.31, S1.40, S1.49, S1.6
- net F': now also S1.16, S1.25, S1.30, S1.39, S1.48, S1.7
- net G': now also S1.17, S1.26, S1.29, S1.38, S1.47, S1.8
- net GND: now also C6.2
- net PIC_A: now also IC1.29 (RD6); no longer IC1.30 (RD7)
- net PIC_B: now also IC1.28 (RD5); no longer IC1.29 (RD6)
- net PIC_C: now also IC1.27 (RD4); no longer IC1.28 (RD5)
- net PIC_D: now also IC1.26 (RC7); no longer IC1.27 (RD4)
- net PIC_DP: now also IC1.30 (RD7); no longer IC1.33 (RB0)
- net PIC_E: now also IC1.25 (RC6); no longer IC1.26 (RC7)
- net PIC_F: now also IC1.24 (RC5); no longer IC1.25 (RC6)
- net PIC_G: now also IC1.22 (RD3); no longer IC1.24 (RC5)
- net at Q6.1 (C): now also S1.54
- net at Q4.1 (C): now also S1.45
- net at Q3.1 (C): now also S1.10
- net at Q2.1 (C): now also S1.36
- net at Q1.1 (C): now also S1.19
- net at Q5.1 (C): now also S1.1
- net MCLR: no longer names the net of IC1.1 (~{MCLR}/VPP/RE3)
- net MCLR: now also R14.1; no longer J7.1
- new net: C6.1, R13.1, R14.2
- new net: J7.1, R13.2

Commit message: backup update
Connections:
- net A_1: now also IC1.33 (RB0); no longer IC1.21 (RD2)
- net A_2: now also IC1.34 (RB1); no longer IC1.17 (RC2)
- net A_3: now also IC1.35 (RB2); no longer IC1.16 (RC1)
- net A_4: now also IC1.36 (RB3); no longer IC1.15 (RC0)
- net A_5: now also IC1.37 (RB4); no longer IC1.14 (RA6)
- net A_6: now also IC1.38 (RB5); no longer IC1.13 (RA7)
- net at Q6.1 (C): now also S1.19; no longer S1.54
- net at Q4.1 (C): now also S1.10; no longer S1.45
- net at Q2.1 (C): now also S1.1; no longer S1.36
- net at Q3.1 (C): now also S1.45; no longer S1.10
- net at Q5.1 (C): now also S1.36; no longer S1.1
- net at Q1.1 (C): now also S1.54; no longer S1.19

Commit message: backup update
Parts:
- added C7, C8: 100uF, Capacitor_THT:CP_Radial_D6.3mm_P2.50mm, symbol Device:C_Small
- C1, C2: footprint Capacitor_SMD:C_0603_1608Metric_Pad1.08x0.95mm_HandSolder -> Capacitor_SMD:C_0805_2012Metric_Pad1.18x1.45mm_HandSolder
Connections:
- net GND: now also C7.1, C8.1
- net VCC: now also C7.2, C8.2

Commit message: backup update
Parts:
- added D1: M7 SMD T/R, Diode_SMD:D_SMA_Handsoldering, symbol Device:D_Small
Connections:
- net GND: now also D1.2 (A); no longer J1.1
- new net: D1.1 (K), J1.1
Other:
- moved on the sheet: C7, C8
