File: Ročníkový projekt S3E.kicad_sch (KiCad schematic)
At the start: 40 parts, among them IC1 PIC18F47Q43-I_P, IC3 ULN2804A, IC5 MCP7940M-I_SN, J1 DG126-5.0-02P-14-00A, J2 - nastavení času, J3 + nastavení času, J7 TSW-105-07-G-S, J8 přepínání mezi číslicemi, Q1 DTA123JCAT116, Q2 DTA123JCAT116, Q3 DTA123JCAT116, Q4 DTA123JCAT116, Q5 DTA123JCAT116, Q6 DTA123JCAT116, Y1 32.768kHz

Commit message: backup update
Connections:
- net A': now also S1.21, S1.36, S1.45; no longer S1.20, S1.35, S1.44, S1.53
- net B': now also S1.22, S1.35, S1.44; no longer S1.21, S1.34, S1.43, S1.52
- net C': now also S1.23, S1.34, S1.43; no longer S1.22, S1.33, S1.42, S1.51
- net D': now also S1.24, S1.33, S1.42; no longer S1.23, S1.32, S1.41, S1.50
- net DP': now also S1.29, S1.38; no longer S1.27, S1.37, S1.46
- net E': now also S1.25, S1.32, S1.41; no longer S1.24, S1.31, S1.40, S1.49
- net F': now also S1.26, S1.31, S1.40; no longer S1.25, S1.30, S1.39, S1.48
- net G': now also S1.27, S1.30, S1.39; no longer S1.26, S1.29, S1.38, S1.47
- net at Q6.1 (C): now also S1.20; no longer S1.19
- net at Q3.1 (C): now also S1.37; no longer S1.45
- net at Q5.1 (C): now also S1.19; no longer S1.36
- net at Q1.1 (C): now also S1.46; no longer S1.54

Commit message: backup update
Parts:
- IC5: footprint SamacSys_Parts:SOIC127P600X175-8N -> SOIC127P600X175-8N

Commit message: backup update
Parts:
- removed C7, C8: 100uF, Capacitor_THT:CP_Radial_D6.3mm_P2.50mm, symbol Device:C_Small
- added C10, C9: 100nF, Capacitor_SMD:C_1206_3216Metric_Pad1.33x1.80mm_HandSolder, symbol Device:C_Small
- added C7, C8: 100uF, Capacitor_THT:CP_Radial_D6.3mm_P2.50mm, symbol Device:C_Polarized_Small
- added IC2: L7805CD2T-TR, My parts:L7805CD2T, symbol My_parts:L7805CD2T-TR
- IC5: footprint SOIC127P600X175-8N -> My parts:SOIC127P600X175-8N
Connections:
- net GND: now also C10.2, C7.2, C8.2, C9.2, IC2.2 (GND)
- net VCC: now also C10.1, IC2.3 (OUTPUT); no longer J1.2
- net at J1.1: now also C7.1, C8.1, C9.1, IC2.1 (INPUT); no longer D1.1 (K)
- new net: D1.1 (K), J1.2
Other:
- moved on the sheet: D1, J1

Commit message: backup update
Parts:
- removed S1: S, My parts:Screen_connector_footprint_parraler, symbol My_parts:Screen_connector_symbol
- added Conn1: ~, My parts:DIP-14_IDC_2x14, symbol My_parts:Connector_IDC_2x7
- C1, C2: value 7pF -> C_Small
- C10, C3, C4, C5, C6, C9: value 100nF -> C_Small
- C7, C8: value 100uF -> C_Polarized_Small
- D1: value M7 SMD T/R -> D_Small
- IC5: footprint My parts:SOIC127P600X175-8N -> SOIC127P600X175-8N
- J2: value - nastavení času -> DS1021-1_2SF11-B
- J3: value + nastavení času -> DS1021-1_2SF11-B
- J8: value přepínání mezi číslicemi -> DS1021-1_2SF11-B
- R1, R13, R19, R2, R3, R4: value 4.7k -> R_Small
- R10, R11, R12, R5, R6, R7, R8, R9: value 330ohm -> R_Small
- R14: value 470R -> R_Small
- Y1: value 32.768kHz -> Crystal_Small
Connections:
- net A: now also IC3.18 (OUT1); no longer IC3.11 (OUT8)
- net A': now also Conn1.12
- net A_1: now also Q6.2 (B); no longer Q2.2 (B)
- net A_2: now also Q5.2 (B); no longer Q1.2 (B)
- net A_5: now also Q2.2 (B); no longer Q6.2 (B)
- net A_6: now also Q1.2 (B); no longer Q5.2 (B)
- net B: now also IC3.17 (OUT2); no longer IC3.12 (OUT7)
- net B': now also Conn1.13
- net C: now also IC3.16 (OUT3); no longer IC3.13 (OUT6)
- net C': now also Conn1.14
- net D: now also IC3.15 (OUT4); no longer IC3.14 (OUT5)
- net D': now also Conn1.11
- net DP: now also IC3.11 (OUT8); no longer IC3.18 (OUT1)
- net DP': now also Conn1.7
- net E: now also IC3.14 (OUT5); no longer IC3.15 (OUT4)
- net E': now also Conn1.10
- net F: now also IC3.13 (OUT6); no longer IC3.16 (OUT3)
- net F': now also Conn1.9
- net G: now also IC3.12 (OUT7); no longer IC3.17 (OUT2)
- net G': now also Conn1.8
- net PIC_A: now also IC1.24 (RC5), IC3.7 (IN7); no longer IC1.29 (RD6), IC3.2 (IN2)
- net PIC_B: now also IC1.25 (RC6), IC3.6 (IN6); no longer IC1.28 (RD5), IC3.3 (IN3)
- net PIC_C: now also IC1.26 (RC7), IC3.5 (IN5); no longer IC1.27 (RD4), IC3.4 (IN4)
- net PIC_D: now also IC1.27 (RD4), IC3.4 (IN4); no longer IC1.26 (RC7), IC3.5 (IN5)
- net PIC_DP: now also IC1.22 (RD3), IC3.8 (IN8); no longer IC1.30 (RD7), IC3.1 (IN1)
- net PIC_E: now also IC1.28 (RD5), IC3.3 (IN3); no longer IC1.25 (RC6), IC3.6 (IN6)
- net PIC_F: now also IC1.29 (RD6), IC3.2 (IN2); no longer IC1.24 (RC5), IC3.7 (IN7)
- net PIC_G: now also IC1.30 (RD7), IC3.1 (IN1); no longer IC1.22 (RD3), IC3.8 (IN8)
- net DIGIT_1: now reaches Q6.1 (C)
- net DIGIT_1: now also Conn1.6
- net DIGIT_3: now reaches Q4.1 (C)
- net DIGIT_3: now also Conn1.4
- net DIGIT_5: now reaches Q2.1 (C)
- net DIGIT_5: now also Conn1.2
- net DIGIT_2: now reaches Q5.1 (C)
- net DIGIT_2: now also Conn1.5
- net DIGIT_4: now reaches Q3.1 (C)
- net DIGIT_4: now also Conn1.3
- net DIGIT_6: now reaches Q1.1 (C)
- net DIGIT_6: now also Conn1.1
Other:
- added sheet Display_Board (Display_Board.kicad_sch)
- moved on the sheet: Q1, Q2, Q3, Q4, Q5, Q6

Commit message: backup update
Parts:
- C1: renamed from C6; value C_Small -> 100nF
- C10, C9: value C_Small -> 100nF
- C2: renamed from C5; value C_Small -> 100nF
- C3: renamed from C4; value C_Small -> 100nF
- C4: renamed from C3; value C_Small -> 100nF
- C5: renamed from C1; value C_Small -> 7pF
- C6: renamed from C2; value C_Small -> 7pF
- C7, C8: value C_Polarized_Small -> 100uF
- D1: value D_Small -> M7 SMD T/R
- R1: renamed from R13; value R_Small -> 4K7
- R10: renamed from R8; value R_Small -> 330R
- R11: renamed from R7; value R_Small -> 330R
- R12: renamed from R6; value R_Small -> 330R
- R13: renamed from R5; value R_Small -> 330R
- R14: renamed from R2; value R_Small -> 4K7
- R15: renamed from R1; value R_Small -> 4k7
- R2: renamed from R14; value R_Small -> 470R
- R3: renamed from R4; value R_Small -> 4K7
- R4: renamed from R3; value R_Small -> 4K7
- R5: renamed from R19; value R_Small -> 4K7
- R6: renamed from R12; value R_Small -> 330R
- R7: renamed from R11; value R_Small -> 330R
- R8: renamed from R10; value R_Small -> 330R
- R9: value R_Small -> 330R
- Y1: value Crystal_Small -> 32 768Hz
- renumbered IC3 to IC2, IC5 to IC3, IC2 to IC4, J7 to J1, J8 to J4, J1 to J5, Q6 to Q1, Q5 to Q2, Q4 to Q3, Q3 to Q4, Q2 to Q5, Q1 to Q6
Connections:
- net Buttons_board/Button_2: now reaches IC1.3 (RA1), J3.2, R4.1
- net Buttons_board/Button_3: now reaches IC1.4 (RA2), J4.2, R5.1
- net Buttons_board/Button_1: now reaches IC1.2 (RA0), J2.2, R3.1
Other:
- added sheet Buttons_board (Buttons.kicad_sch)
