File: Ročníkový projekt S3E.kicad_sch (KiCad schematic)
At the start: 43 parts, among them IC1 PIC18F47Q43-I_P, IC2 ULN2804A, IC3 MCP7940M-I_SN, IC4 L7805CD2T-TR, J1 TSW-105-07-G-S, J2 DS1021-1_2SF11-B, J3 DS1021-1_2SF11-B, J4 DS1021-1_2SF11-B, J5 DG126-5.0-02P-14-00A, Q1 DTA123JCAT116, Q2 DTA123JCAT116, Q3 DTA123JCAT116, Q4 DTA123JCAT116, Q5 DTA123JCAT116, Q6 DTA123JCAT116, Y1 32 768Hz

Commit message: Auto-backup: 21:43:30 13/04/2026
Parts:
- R15: value 4k7 -> 4K7
- renumbered C8 to C1, C4 to C10, C7 to C2, C9 to C3, C10 to C4, C1 to C5, C3 to C6, C2 to C7, C6 to C8, C5 to C9, IC4 to IC3, IC3 to IC4, J5 to J1, J1 to J4, J4 to J5, Q2 to Q1, Q4 to Q2, Q6 to Q4, Q1 to Q6, R9 to R1, R2 to R10, R3 to R11, R1 to R12, R5 to R13, R6 to R2, R10 to R3, R8 to R4, R7 to R5, R11 to R6, R12 to R7, R13 to R8, R4 to R9
Changed lines of the file:
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@@
 		(on_board yes)
 		(dnp no)
-		(property "Reference" "Q1"
+		(property "Reference" "Q6"
 			(at 227.33 213.3599 0)
 			(effects
@@
 			(project "Ročníkový projekt S3E"
 				(path "/c4e08560-2444-47e9-8324-16df61887a86"
-					(reference "Q1")
+					(reference "Q6")
 					(unit 1)
 				)
@@
 		(on_board yes)
 		(dnp no)
-		(property "Reference" "R4"
+		(property "Reference" "R9"
 			(at 62.992 72.136 90)
 			(effects
@@
 			(project ""
 				(path "/c4e08560-2444-47e9-8324-16df61887a86"
-					(reference "R4")
+					(reference "R9")
 					(unit 1)
 				)
@@
 		(dnp no)
 		(fields_autoplaced yes)
-		(property "Reference" "C4"
+		(property "Reference" "C10"
 			(at 55.88 160.0262 0)
 			(effects
@@
 			(project ""
 				(path "/c4e08560-2444-47e9-8324-16df61887a86"
-					(reference "C4")
+					(reference "C10")
 					(unit 1)
 				)
@@
 		(on_board yes)
 		(dnp no)
-		(property "Reference" "R5"
+		(property "Reference" "R13"
 			(at 64.262 94.996 90)
 			(effects
@@
 			(project "Ročníkový projekt S3E"
 				(path "/c4e08560-2444-47e9-8324-16df61887a86"
-					(reference "R5")
+					(reference "R13")
 					(unit 1)
 				)
@@
 		(on_board yes)
 		(dnp no)
-		(property "Reference" "R2"
+		(property "Reference" "R10"
 			(at 145.796 47.498 0)
 			(effects
@@
 			(project "Ročníkový projekt S3E"
 				(path "/c4e08560-2444-47e9-8324-16df61887a86"
-					(reference "R2")
+					(reference "R10")
 					(unit 1)
 				)
@@
 		(on_board yes)
 		(dnp no)
-		(property "Reference" "R3"
+		(property "Reference" "R11"
 			(at 62.738 51.816 90)
 			(effects
@@
 			(project "Ročníkový projekt S3E"
 				(path "/c4e08560-2444-47e9-8324-16df61887a86"
-					(reference "R3")
+					(reference "R11")
 					(unit 1)
 				)
@@
 		(on_board yes)
 		(dnp no)
-		(property "Reference" "C5"
+		(property "Reference" "C9"
 			(at 19.304 172.72 0)
 			(effects
@@
 			(project "Ročníkový projekt S3E"
 				(path "/c4e08560-2444-47e9-8324-16df61887a86"
-					(reference "C5")
+					(reference "C9")
 					(unit 1)
 				)
@@
 		(on_board yes)
 		(dnp no)
-		(property "Reference" "R13"
+		(property "Reference" "R8"
 			(at 365.76 126.9999 0)
 			(effects
@@
 			(project ""
 				(path "/c4e08560-2444-47e9-8324-16df61887a86"
-					(reference "R13")
+					(reference "R8")
 					(unit 1)
 				)
@@
 		(on_board yes)
 		(dnp no)
-		(property "Reference" "C3"
+		(property "Reference" "C6"
 			(at 127.508 82.042 0)
 			(effects
@@
 			(project ""
 				(path "/c4e08560-2444-47e9-8324-16df61887a86"
-					(reference "C3")
+					(reference "C6")
 					(unit 1)
 				)
@@
 		(dnp no)
 		(fields_autoplaced yes)
-		(property "Reference" "IC3"
+		(property "Reference" "IC4"
 			(at 68.58 142.24 0)
 			(effects
@@
 			(project ""
 				(path "/c4e08560-2444-47e9-8324-16df61887a86"
-					(reference "IC3")
+					(reference "IC4")
 					(unit 1)
 				)
@@
 		(dnp no)
 		(fields_autoplaced yes)
-		(property "Reference" "R11"
+		(property "Reference" "R6"
 			(at 342.9 126.9999 0)
 			(effects
@@
 			(project "Ročníkový projekt S3E"
 				(path "/c4e08560-2444-47e9-8324-16df61887a86"
-					(reference "R11")
+					(reference "R6")
 					(unit 1)
 				)
@@
 		(dnp no)
 		(fields_autoplaced yes)
-		(property "Reference" "R7"
+		(property "Reference" "R5"
 			(at 297.18 126.9999 0)
 			(effects
@@
 			(project "Ročníkový projekt S3E"
 				(path "/c4e08560-2444-47e9-8324-16df61887a86"
-					(reference "R7")
+					(reference "R5")
 					(unit 1)
 				)
@@
 		(dnp no)
 		(fields_autoplaced yes)
-		(property "Reference" "J1"
+		(property "Reference" "J4"
 			(at 173.99 20.3199 90)
 			(effects
@@
 			(project ""
 				(path "/c4e08560-2444-47e9-8324-16df61887a86"
-					(reference "J1")
+					(reference "J4")
 					(unit 1)
 				)
@@
 		(on_board yes)
 		(dnp no)
-		(property "Reference" "J4"
+		(property "Reference" "J5"
 			(at 50.546 105.664 90)
 			(effects
@@
 			(project "Ročníkový projekt S3E"
 				(path "/c4e08560-2444-47e9-8324-16df61887a86"
-					(reference "J4")
+					(reference "J5")
 					(unit 1)
 				)
@@
 			)
 		)
-		(property "Value" "4k7"
+		(property "Value" "4K7"
 			(at 96.266 164.084 0)
 			(effects
@@
 		(dnp no)
 		(fields_autoplaced yes)
-		(property "Reference" "C6"
+		(property "Reference" "C8"
 			(at 36.83 172.7135 0)
 			(effects
@@
 			(project ""
 				(path "/c4e08560-2444-47e9-8324-16df61887a86"
-					(reference "C6")
+					(reference "C8")
 					(unit 1)
 				)
@@
 		(on_board yes)
 		(dnp no)
-		(property "Reference" "C9"
+		(property "Reference" "C3"
 			(at 63.246 216.154 90)
 			(effects
@@
 			(project ""
 				(path "/c4e08560-2444-47e9-8324-16df61887a86"
-					(reference "C9")
+					(reference "C3")
 					(unit 1)
 				)
@@
 		(on_board yes)
 		(dnp no)
-		(property "Reference" "Q4"
+		(property "Reference" "Q2"
 			(at 283.21 213.3599 0)
 			(effects
@@
 			(project "Ročníkový projekt S3E"
 				(path "/c4e08560-2444-47e9-8324-16df61887a86"
-					(reference "Q4")
+					(reference "Q2")
 					(unit 1)
 				)
@@
 		(on_board yes)
 		(dnp no)
-		(property "Reference" "C7"
+		(property "Reference" "C2"
 			(at 57.8739 200.66 90)
 			(effects
@@
 			(project ""
 				(path "/c4e08560-2444-47e9-8324-16df61887a86"
-					(reference "C7")
+					(reference "C2")
 					(unit 1)
 				)
@@
 		(on_board yes)
 		(dnp no)
-		(property "Reference" "C10"
+		(property "Reference" "C4"
 			(at 58.166 237.998 90)
 			(effects
@@
 			(project "Ročníkový projekt S3E"
 				(path "/c4e08560-2444-47e9-8324-16df61887a86"
-					(reference "C10")
+					(reference "C4")
 					(unit 1)
 				)
@@
 		(on_board yes)
 		(dnp no)
-		(property "Reference" "R1"
+		(property "Reference" "R12"
 			(at 132.334 37.338 0)
 			(effects
@@
 			(project "Ročníkový projekt S3E"
 				(path "/c4e08560-2444-47e9-8324-16df61887a86"
-					(reference "R1")
+					(reference "R12")
 					(unit 1)
 				)
@@
 		(dnp no)
 		(fields_autoplaced yes)
-		(property "Reference" "R9"
+		(property "Reference" "R1"
 			(at 320.04 126.9999 0)
 			(effects
@@
 			(project "Ročníkový projekt S3E"
 				(path "/c4e08560-2444-47e9-8324-16df61887a86"
-					(reference "R9")
+					(reference "R1")
 					(unit 1)
 				)
@@
 		(on_board yes)
 		(dnp no)
-		(property "Reference" "C1"
+		(property "Reference" "C5"
 			(at 134.62 41.9162 0)
 			(effects
@@
 			(project "Ročníkový projekt S3E"
 				(path "/c4e08560-2444-47e9-8324-16df61887a86"
-					(reference "C1")
+					(reference "C5")
 					(unit 1)
 				)
@@
 		(dnp no)
 		(fields_autoplaced yes)
-		(property "Reference" "R10"
+		(property "Reference" "R3"
 			(at 331.47 126.9999 0)
 			(effects
@@
 			(project "Ročníkový projekt S3E"
 				(path "/c4e08560-2444-47e9-8324-16df61887a86"
-					(reference "R10")
+					(reference "R3")
 					(unit 1)
 				)
@@
 		(dnp no)
 		(fields_autoplaced yes)
-		(property "Reference" "R12"
+		(property "Reference" "R7"
 			(at 354.33 126.9999 0)
 			(effects
@@
 			(project "Ročníkový projekt S3E"
 				(path "/c4e08560-2444-47e9-8324-16df61887a86"
-					(reference "R12")
+					(reference "R7")
 					(unit 1)
 				)
@@
 		(dnp no)
 		(fields_autoplaced yes)
-		(property "Reference" "R8"
+		(property "Reference" "R4"
 			(at 308.61 126.9999 0)
 			(effects
@@
 			(project "Ročníkový projekt S3E"
 				(path "/c4e08560-2444-47e9-8324-16df61887a86"
-					(reference "R8")
+					(reference "R4")
 					(unit 1)
 				)
@@
 		(dnp no)
 		(fields_autoplaced yes)
-		(property "Reference" "R6"
+		(property "Reference" "R2"
 			(at 285.75 126.9999 0)
 			(effects
@@
 			(project "Ročníkový projekt S3E"
 				(path "/c4e08560-2444-47e9-8324-16df61887a86"
-					(reference "R6")
+					(reference "R2")
 					(unit 1)
 				)
@@
 		(on_board yes)
 		(dnp no)
-		(property "Reference" "C8"
+		(property "Reference" "C1"
 			(at 55.626 214.122 90)
 			(effects
@@
 			(project "Ročníkový projekt S3E"
 				(path "/c4e08560-2444-47e9-8324-16df61887a86"
-					(reference "C8")
+					(reference "C1")
 					(unit 1)
 				)
@@
 		(dnp no)
 		(fields_autoplaced yes)
-		(property "Reference" "J5"
+		(property "Reference" "J1"
 			(at 63.5 189.2299 90)
 			(effects
@@
 			(project ""
 				(path "/c4e08560-2444-47e9-8324-16df61887a86"
-					(reference "J5")
+					(reference "J1")
 					(unit 1)
 				)
@@
 		(on_board yes)
 		(dnp no)
-		(property "Reference" "Q2"
+		(property "Reference" "Q1"
 			(at 246.38 213.3599 0)
 			(effects
@@
 			(project "Ročníkový projekt S3E"
 				(path "/c4e08560-2444-47e9-8324-16df61887a86"
-					(reference "Q2")
+					(reference "Q1")
 					(unit 1)
 				)
@@
 		(on_board yes)
 		(dnp no)
-		(property "Reference" "IC4"
+		(property "Reference" "IC3"
 			(at 34.036 227.838 0)
 			(effects
@@
 			(project ""
 				(path "/c4e08560-2444-47e9-8324-16df61887a86"
-					(reference "IC4")
+					(reference "IC3")
 					(unit 1)
 				)
@@
 		(on_board yes)
 		(dnp no)
-		(property "Reference" "Q6"
+		(property "Reference" "Q4"
 			(at 323.85 213.3599 0)
 			(effects
@@
 			(project ""
 				(path "/c4e08560-2444-47e9-8324-16df61887a86"
-					(reference "Q6")
+					(reference "Q4")
 					(unit 1)
 				)
@@
 		(on_board yes)
 		(dnp no)
-		(property "Reference" "C2"
+		(property "Reference" "C7"
 			(at 219.456 76.962 0)
 			(effects
@@
 			(project ""
 				(path "/c4e08560-2444-47e9-8324-16df61887a86"
-					(reference "C2")
+					(reference "C7")
 					(unit 1)
 				)

Commit message: Auto-backup: 09:05:42 15/04/2026
Parts:
- Conn1: value ~ -> (none)

Commit message: Auto-backup: 10:53:27 17/04/2026
Parts:
- removed C10: 100nF, Capacitor_SMD:C_1206_3216Metric_Pad1.33x1.80mm_HandSolder, symbol Device:C_Small
- removed IC2: ULN2804A, My parts:DIP850W46P254L2324H393Q18N, symbol My_parts:ULN2804A
- removed Q1, Q2, Q3, Q4, Q5, Q6: DTA123JCAT116, My parts:TRANS_DTA113ZCAH_ROM, symbol My_parts:DTA123JCAT116
- added C4: 100nF, Capacitor_SMD:C_1206_3216Metric_Pad1.33x1.80mm_HandSolder, symbol Device:C_Small
- added Q1, Q2, Q3, Q4, Q5, Q6: YJL2301D, My parts:SOT95P240X115-3N, symbol My_parts:YJL2301D
- added R16, R17, R18, R19, R20, R21: 10K, Resistor_SMD:R_0805_2012Metric_Pad1.20x1.40mm_HandSolder, symbol Device:R_Small
- added U1: ULN2803A, Package_DIP:DIP-18_W7.62mm, symbol Transistor_Array:ULN2803A
- C5: renamed from C9; value 7pF -> 6,8pF
- C6: renamed from C8; value 7pF -> 6,8pF
- IC2: renamed from IC4; footprint SOIC127P600X175-8N -> My parts:SOIC127P600X175-8N
- R10: renamed from R3; value 330R -> 220R; footprint Resistor_THT:R_Axial_DIN0309_L9.0mm_D3.2mm_P12.70mm_Horizontal -> Resistor_SMD:R_1206_3216Metric_Pad1.30x1.75mm_HandSolder
- R11: renamed from R6; value 330R -> 220R; footprint Resistor_THT:R_Axial_DIN0309_L9.0mm_D3.2mm_P12.70mm_Horizontal -> Resistor_SMD:R_1206_3216Metric_Pad1.30x1.75mm_HandSolder
- R12: renamed from R7; value 330R -> 220R; footprint Resistor_THT:R_Axial_DIN0309_L9.0mm_D3.2mm_P12.70mm_Horizontal -> Resistor_SMD:R_1206_3216Metric_Pad1.30x1.75mm_HandSolder
- R13: renamed from R8; value 330R -> 220R; footprint Resistor_THT:R_Axial_DIN0309_L9.0mm_D3.2mm_P12.70mm_Horizontal -> Resistor_SMD:R_1206_3216Metric_Pad1.30x1.75mm_HandSolder
- R6: renamed from R2; value 330R -> 220R; footprint Resistor_THT:R_Axial_DIN0309_L9.0mm_D3.2mm_P12.70mm_Horizontal -> Resistor_SMD:R_1206_3216Metric_Pad1.30x1.75mm_HandSolder
- R7: renamed from R5; value 330R -> 220R; footprint Resistor_THT:R_Axial_DIN0309_L9.0mm_D3.2mm_P12.70mm_Horizontal -> Resistor_SMD:R_1206_3216Metric_Pad1.30x1.75mm_HandSolder
- R8: renamed from R4; value 330R -> 220R; footprint Resistor_THT:R_Axial_DIN0309_L9.0mm_D3.2mm_P12.70mm_Horizontal -> Resistor_SMD:R_1206_3216Metric_Pad1.30x1.75mm_HandSolder
- R9: renamed from R1; value 330R -> 220R; footprint Resistor_THT:R_Axial_DIN0309_L9.0mm_D3.2mm_P12.70mm_Horizontal -> Resistor_SMD:R_1206_3216Metric_Pad1.30x1.75mm_HandSolder
- renumbered C5 to C1, C4 to C10, C7 to C2, C6 to C3, C2 to C7, C1 to C8, C3 to C9, J4 to J1, J5 to J4, J1 to J5, R12 to R1, R10 to R2, R11 to R3, R9 to R4, R13 to R5
Connections:
- net A: now also U1.12 (O7)
- net A': now also Conn1.13; no longer Conn1.12
- net A_1: now also Q1.1 (G), R16.2
- net A_2: now also Q2.1 (G), R17.2
- net A_3: now also Q3.1 (G), R18.2
- net A_4: now also Q4.1 (G), R19.2
- net A_5: now also Q5.1 (G), R20.2
- net A_6: now also Q6.1 (G), R21.2
- net B: now also U1.13 (O6)
- net B': now also Conn1.12; no longer Conn1.13
- net C: now also U1.14 (O5)
- net C': now also Conn1.11; no longer Conn1.14
- net D: now also U1.15 (O4)
- net D': now also Conn1.10; no longer Conn1.11
- net DP: now also U1.11 (O8)
- net DP': now also Conn1.14; no longer Conn1.7
- net E: now also U1.16 (O3)
- net E': now also Conn1.9; no longer Conn1.10
- net F: now also U1.17 (O2)
- net F': now also Conn1.8; no longer Conn1.9
- net G: now also U1.18 (O1)
- net G': now also Conn1.7; no longer Conn1.8
- net GND: now also IC2.4 (VSS), C4.2, U1.9 (GND); no longer IC2.8 (VCC)
- net PIC_A: now also U1.7 (I7)
- net PIC_B: now also U1.6 (I6)
- net PIC_C: now also U1.5 (I5)
- net PIC_D: now also U1.4 (I4)
- net PIC_DP: now also U1.8 (I8)
- net PIC_E: now also U1.3 (I3)
- net PIC_F: now also U1.2 (I2)
- net PIC_G: now also U1.1 (I1)
- net VCC: now also IC2.8 (VCC), C4.1, Q1.2 (S), Q2.2 (S), Q3.2 (S), Q4.2 (S), Q5.2 (S), Q6.2 (S), R16.1, R17.1, R18.1, R19.1, R20.1, R21.1, U1.10 (COM); no longer IC2.4 (VSS)
- net DIGIT_1 renamed Display_Board/D1
- net Display_Board/D1: now also Q1.3 (D)
- net DIGIT_2 renamed Display_Board/D2
- net Display_Board/D2: now also Q2.3 (D)
- net DIGIT_3 renamed Display_Board/D3
- net Display_Board/D3: now also Q3.3 (D)
- net DIGIT_4 renamed Display_Board/D4
- net Display_Board/D4: now also Q4.3 (D)
- net DIGIT_5 renamed Display_Board/D5
- net Display_Board/D5: now also Q5.3 (D)
- net DIGIT_6 renamed Display_Board/D6
- net Display_Board/D6: now also Q6.3 (D)
Other:
- sheet Display_Board ports: added A, B, C, D, D1, D2, D3, D4, D5, D6, DP, E, F, G; removed none

Commit message: Auto-backup: 15:10:38 17/04/2026
Other:
- moved on the sheet: R3
Changed lines of the file:
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@@
 	)
 	(junction
+		(at 66.04 54.61)
+		(diameter 0)
+		(color 0 0 0 0)
+	)
+	(junction
 		(at 283.21 219.71)
 		(diameter 0)
@@
 	)
 	(junction
-		(at 73.66 243.84)
-		(diameter 0)
-		(color 0 0 0 0)
-	)
-	(junction
 		(at 43.18 212.09)
 		(diameter 0)
@@
 	)
 	(junction
-		(at 43.18 243.84)
-		(diameter 0)
-		(color 0 0 0 0)
-	)
-	(junction
 		(at 327.66 134.62)
 		(diameter 0)
@@
 	)
 	(junction
-		(at 66.04 54.61)
-		(diameter 0)
-		(color 0 0 0 0)
-	)
-	(junction
 		(at 186.69 181.61)
 		(diameter 0)
@@
 	(wire
 		(pts
-			(xy 40.64 243.84) (xy 43.18 243.84)
-		)
-		(stroke
-			(width 0)
-			(type default)
-		)
-	)
-	(wire
-		(pts
 			(xy 317.5 123.19) (xy 317.5 125.73)
 		)
@@
 	(wire
 		(pts
-			(xy 71.12 243.84) (xy 73.66 243.84)
-		)
-		(stroke
-			(width 0)
-			(type default)
-		)
-	)
-	(wire
-		(pts
 			(xy 360.68 215.9) (xy 374.65 215.9)
 		)
@@
 	(wire
 		(pts
+			(xy 63.5 54.61) (xy 66.04 54.61)
+		)
+		(stroke
+			(width 0)
+			(type default)
+		)
+	)
+	(wire
+		(pts
 			(xy 320.04 71.12) (xy 325.12 71.12)
 		)
@@
 		)
 	)
-	(global_label "VCC_P"
-		(shape input)
-		(at 162.56 31.75 270)
-		(fields_autoplaced yes)
-		(effects
-			(font
-				(size 1.27 1.27)
-			)
-			(justify right)
-		)
-		(property "Intersheetrefs" "${INTERSHEET_REFS}"
-			(at 162.56 40.6014 90)
-			(hide yes)
-			(show_name no)
-			(do_not_autoplace no)
-			(effects
-				(font
-					(size 1.27 1.27)
-				)
-				(justify right)
-			)
-		)
-	)
 	(global_label "PIC_B"
 		(shape input)
@@
 		)
 	)
-	(global_label "VCC_P"
-		(shape input)
-		(at 40.64 243.84 180)
-		(fields_autoplaced yes)
-		(effects
-			(font
-				(size 1.27 1.27)
-			)
-			(justify right)
-		)
-		(property "Intersheetrefs" "${INTERSHEET_REFS}"
-			(at 31.7886 243.84 0)
-			(hide yes)
-			(show_name no)
-			(do_not_autoplace no)
-			(effects
-				(font
-					(size 1.27 1.27)
-				)
-				(justify right)
-			)
-		)
-	)
 	(global_label "A_6"
 		(shape input)
@@
 		)
 	)
-	(global_label "VDD_P"
-		(shape input)
-		(at 71.12 243.84 180)
-		(fields_autoplaced yes)
-		(effects
-			(font
-				(size 1.27 1.27)
-			)
-			(justify right)
-		)
-		(property "Intersheetrefs" "${INTERSHEET_REFS}"
-			(at 62.2686 243.84 0)
-			(hide yes)
-			(show_name no)
-			(do_not_autoplace no)
-			(effects
-				(font
-					(size 1.27 1.27)
-				)
-				(justify right)
-			)
-		)
-	)
 	(global_label "A_5"
 		(shape input)
@@
 		)
 	)
-	(global_label "VDD_P"
-		(shape input)
-		(at 165.1 31.75 270)
-		(fields_autoplaced yes)
-		(effects
-			(font
-				(size 1.27 1.27)
+	(symbol
+		(lib_id "power:VCC")
+		(at 162.56 31.75 180)
+		(unit 1)
+		(body_style 1)
+		(exclude_from_sim no)
+		(in_bom yes)
+		(on_board yes)
+		(in_pos_files yes)
+		(dnp no)
+		(property "Reference" "#PWR033"
+			(at 162.56 27.94 0)
+			(hide yes)
+			(show_name no)
+			(do_not_autoplace no)
+			(effects
+				(font
+					(size 1.27 1.27)
+				)
 			)
-			(justify right)
 		)
-		(property "Intersheetrefs" "${INTERSHEET_REFS}"
-			(at 165.1 40.6014 90)
-			(hide yes)
+		(property "Value" "VCC"
+			(at 158.75 35.56 0)
 			(show_name no)
 			(do_not_autoplace no)
@@
 			)
 		)
+		(property "Footprint" ""
+			(at 162.56 31.75 0)
+			(hide yes)
+			(show_name no)
+			(do_not_autoplace no)
+			(effects
+				(font
+					(size 1.27 1.27)
+				)
+			)
+		)
+		(property "Datasheet" ""
+			(at 162.56 31.75 0)
+			(hide yes)
+			(show_name no)
+			(do_not_autoplace no)
+			(effects
+				(font
+					(size 1.27 1.27)
+				)
+			)
+		)
+		(property "Description" "Power symbol creates a global label with name \"VCC\""
+			(at 162.56 31.75 0)
+			(hide yes)
+			(show_name no)
+			(do_not_autoplace no)
+			(effects
+				(font
+					(size 1.27 1.27)
+				)
+			)
+		)
+		(pin "1"
+		)
+		(instances
+			(project "Ročníkový projekt S3E"
+				(path "/c4e08560-2444-47e9-8324-16df61887a86"
+					(reference "#PWR033")
+					(unit 1)
+				)
+			)
+		)
 	)
 	(symbol
@@
 	)
 	(symbol
+		(lib_id "power:GND")
+		(at 165.1 31.75 0)
+		(unit 1)
+		(body_style 1)
+		(exclude_from_sim no)
+		(in_bom yes)
+		(on_board yes)
+		(in_pos_files yes)
+		(dnp no)
+		(property "Reference" "#PWR032"
+			(at 165.1 38.1 0)
+			(hide yes)
+			(show_name no)
+			(do_not_autoplace no)
+			(effects
+				(font
+					(size 1.27 1.27)
+				)
+			)
+		)
+		(property "Value" "GND"
+			(at 162.56 35.56 0)
+			(show_name no)
+			(do_not_autoplace no)
+			(effects
+				(font
+					(size 1.27 1.27)
+				)
+				(justify left)
+			)
+		)
+		(property "Footprint" ""
+			(at 165.1 31.75 0)
+			(hide yes)
+			(show_name no)
+			(do_not_autoplace no)
+			(effects
+				(font
+					(size 1.27 1.27)
+				)
+			)
+		)
+		(property "Datasheet" ""
+			(at 165.1 31.75 0)
+			(hide yes)
+			(show_name no)
+			(do_not_autoplace no)
+			(effects
+				(font
+					(size 1.27 1.27)
+				)
+			)
+		)
+		(property "Description" "Power symbol creates a global label with name \"GND\" , ground"
+			(at 165.1 31.75 0)
+			(hide yes)
+			(show_name no)
+			(do_not_autoplace no)
+			(effects
+				(font
+					(size 1.27 1.27)
+				)
+			)
+		)
+		(pin "1"
+		)
+		(instances
+			(project "Ročníkový projekt S3E"
+				(path "/c4e08560-2444-47e9-8324-16df61887a86"
+					(reference "#PWR032")
+					(unit 1)
+				)
+			)
+		)
+	)
+	(symbol
 		(lib_id "My_parts:YJL2301D")
 		(at 179.07 219.71 0)
@@
 	(symbol
 		(lib_id "Device:R_Small")
-		(at 63.5 54.61 270)
+		(at 60.96 54.61 270)
 		(unit 1)
 		(body_style 1)
@@
 		(dnp no)
 		(property "Reference" "R3"
-			(at 62.738 51.816 90)
+			(at 60.198 51.816 90)
 			(show_name no)
 			(do_not_autoplace no)
@@
 		)
 		(property "Value" "4K7"
-			(at 62.23 49.784 90)
+			(at 59.69 49.784 90)
 			(show_name no)
 			(do_not_autoplace no)
@@
 		)
 		(property "Footprint" "Resistor_SMD:R_1206_3216Metric_Pad1.30x1.75mm_HandSolder"
-			(at 63.5 54.61 0)
+			(at 60.96 54.61 0)
 			(hide yes)
 			(show_name no)
@@
 		)
 		(property "Datasheet" ""
-			(at 63.5 54.61 0)
+			(at 60.96 54.61 0)
 			(hide yes)
 			(show_name no)
@@
 		)
 		(property "Description" "Resistor, small symbol"
-			(at 63.5 54.61 0)
+			(at 60.96 54.61 0)
 			(hide yes)
 			(show_name no)
@@
 	(symbol
 		(lib_id "power:GND")
-		(at 60.96 54.61 270)
+		(at 58.42 54.61 270)
 		(unit 1)
 		(body_style 1)
@@
 		(fields_autoplaced yes)
 		(property "Reference" "#PWR02"
-			(at 54.61 54.61 0)
+			(at 52.07 54.61 0)
 			(hide yes)
 			(show_name no)
@@
 		)
 		(property "Value" "GND"
-			(at 55.88 54.61 0)
+			(at 53.34 54.61 0)
 			(show_name no)
 			(do_not_autoplace no)
@@
 		)
 		(property "Footprint" ""
-			(at 60.96 54.61 0)
+			(at 58.42 54.61 0)
 			(hide yes)
 			(show_name no)
@@
 		)
 		(property "Datasheet" ""
-			(at 60.96 54.61 0)
+			(at 58.42 54.61 0)
 			(hide yes)
 			(show_name no)
@@
 		)
 		(property "Description" "Power symbol creates a global label with name \"GND\" , ground"
-			(at 60.96 54.61 0)
+			(at 58.42 54.61 0)
 			(hide yes)
 			(show_name no)

Commit message: Auto-backup: 18:09:10 17/04/2026
Parts:
- IC2: footprint My parts:SOIC127P600X175-8N -> SOIC127P600X175-8N
- Y1: footprint Crystal:32.768KHz Vertical 3_8mm -> My parts:Crystal_C38-LF_D3.0mm_L8.0mm_Vertical MY 32kHz
- renumbered Conn1 to J5, J5 to J6
Connections:
- no-connect marks 0 -> 15
Other:
- moved on the sheet: J5, Q1, Q2, Q3, Q4, Q5, Q6, R10, R11, R12, R13, R16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
