File: Buttons.kicad_sch (KiCad schematic)
At the start: 6 parts, among them J6 DS1021-1_2SF11-B, J7 DS1021-1_2SF11-B, J8 DS1021-1_2SF11-B

Commit message: Auto-backup: 21:43:30 13/04/2026
Parts:
- renumbered J7 to J6, J8 to J7, J6 to J8, S2 to S1, S3 to S2, S4 to S3
Changed lines of the file:
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@@
 		(dnp no)
 		(fields_autoplaced yes)
-		(property "Reference" "J6"
+		(property "Reference" "J8"
 			(at 78.74 76.2 0)
 			(effects
@@
 			(project ""
 				(path "/c4e08560-2444-47e9-8324-16df61887a86/fbd34285-b602-47a7-9c37-182089d835a8"
-					(reference "J6")
+					(reference "J8")
 					(unit 1)
 				)
@@
 		(dnp no)
 		(fields_autoplaced yes)
-		(property "Reference" "S3"
+		(property "Reference" "S2"
 			(at 156.21 76.2 0)
 			(effects
@@
 			(project "Ročníkový projekt S3E"
 				(path "/c4e08560-2444-47e9-8324-16df61887a86/fbd34285-b602-47a7-9c37-182089d835a8"
-					(reference "S3")
+					(reference "S2")
 					(unit 1)
 				)
@@
 		(dnp no)
 		(fields_autoplaced yes)
-		(property "Reference" "S4"
+		(property "Reference" "S3"
 			(at 204.47 76.2 0)
 			(effects
@@
 			(project "Ročníkový projekt S3E"
 				(path "/c4e08560-2444-47e9-8324-16df61887a86/fbd34285-b602-47a7-9c37-182089d835a8"
-					(reference "S4")
+					(reference "S3")
 					(unit 1)
 				)
@@
 		(dnp no)
 		(fields_autoplaced yes)
-		(property "Reference" "J7"
+		(property "Reference" "J6"
 			(at 127 76.2 0)
 			(effects
@@
 			(project "Ročníkový projekt S3E"
 				(path "/c4e08560-2444-47e9-8324-16df61887a86/fbd34285-b602-47a7-9c37-182089d835a8"
-					(reference "J7")
+					(reference "J6")
 					(unit 1)
 				)
@@
 		(dnp no)
 		(fields_autoplaced yes)
-		(property "Reference" "J8"
+		(property "Reference" "J7"
 			(at 175.26 76.2 0)
 			(effects
@@
 			(project "Ročníkový projekt S3E"
 				(path "/c4e08560-2444-47e9-8324-16df61887a86/fbd34285-b602-47a7-9c37-182089d835a8"
-					(reference "J8")
+					(reference "J7")
 					(unit 1)
 				)
@@
 		(dnp no)
 		(fields_autoplaced yes)
-		(property "Reference" "S2"
+		(property "Reference" "S1"
 			(at 107.95 76.2 0)
 			(effects
@@
 			(project ""
 				(path "/c4e08560-2444-47e9-8324-16df61887a86/fbd34285-b602-47a7-9c37-182089d835a8"
-					(reference "S2")
+					(reference "S1")
 					(unit 1)
 				)

Commit message: Auto-backup: 10:53:27 17/04/2026
Parts:
- J6: renamed from J8; footprint HDRV2W64P0X254_1X2_508X254X588P -> SamacSys_Parts:HDRV2W64P0X254_1X2_508X254X588P
- J7: renamed from J6; footprint HDRV2W64P0X254_1X2_508X254X588P -> SamacSys_Parts:HDRV2W64P0X254_1X2_508X254X588P
- J8: renamed from J7; footprint HDRV2W64P0X254_1X2_508X254X588P -> SamacSys_Parts:HDRV2W64P0X254_1X2_508X254X588P
- S4: renamed from S1; footprint TACT67NF -> My parts:TACT67NF
- S5: renamed from S2; footprint TACT67NF -> My parts:TACT67NF
- S6: renamed from S3; footprint TACT67NF -> My parts:TACT67NF
Changed lines of the file:
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@@
+		)
+	)
+	(label ""
+		(at 30.48 82.55 0)
+		(effects
+			(font
+				(size 1.27 1.27)
+			)
+			(justify left bottom)
 		)
 	)
@@
 		(dnp no)
 		(fields_autoplaced yes)
-		(property "Reference" "J8"
+		(property "Reference" "J6"
 			(at 78.74 76.2 0)
 			(show_name no)
@@
 			)
 		)
-		(property "Footprint" "HDRV2W64P0X254_1X2_508X254X588P"
+		(property "Footprint" "SamacSys_Parts:HDRV2W64P0X254_1X2_508X254X588P"
 			(at 72.39 -8.56 0)
 			(hide yes)
@@
 			(project "Ročníkový projekt S3E"
 				(path "/c4e08560-2444-47e9-8324-16df61887a86/fbd34285-b602-47a7-9c37-182089d835a8"
-					(reference "J8")
+					(reference "J6")
 					(unit 1)
 				)
@@
 		(dnp no)
 		(fields_autoplaced yes)
-		(property "Reference" "S2"
+		(property "Reference" "S5"
 			(at 156.21 76.2 0)
 			(show_name no)
@@
 			)
 		)
-		(property "Footprint" "TACT67NF"
+		(property "Footprint" "My parts:TACT67NF"
 			(at 162.56 178.74 0)
 			(hide yes)
@@
 			(project "Ročníkový projekt S3E"
 				(path "/c4e08560-2444-47e9-8324-16df61887a86/fbd34285-b602-47a7-9c37-182089d835a8"
-					(reference "S2")
+					(reference "S5")
 					(unit 1)
 				)
@@
 		(dnp no)
 		(fields_autoplaced yes)
-		(property "Reference" "S3"
+		(property "Reference" "S6"
 			(at 204.47 76.2 0)
 			(show_name no)
@@
 			)
 		)
-		(property "Footprint" "TACT67NF"
+		(property "Footprint" "My parts:TACT67NF"
 			(at 210.82 178.74 0)
 			(hide yes)
@@
 			(project "Ročníkový projekt S3E"
 				(path "/c4e08560-2444-47e9-8324-16df61887a86/fbd34285-b602-47a7-9c37-182089d835a8"
-					(reference "S3")
+					(reference "S6")
 					(unit 1)
 				)
@@
 		(dnp no)
 		(fields_autoplaced yes)
-		(property "Reference" "J6"
+		(property "Reference" "J7"
 			(at 127 76.2 0)
 			(show_name no)
@@
 			)
 		)
-		(property "Footprint" "HDRV2W64P0X254_1X2_508X254X588P"
+		(property "Footprint" "SamacSys_Parts:HDRV2W64P0X254_1X2_508X254X588P"
 			(at 120.65 -8.56 0)
 			(hide yes)
@@
 			(project "Ročníkový projekt S3E"
 				(path "/c4e08560-2444-47e9-8324-16df61887a86/fbd34285-b602-47a7-9c37-182089d835a8"
-					(reference "J6")
+					(reference "J7")
 					(unit 1)
 				)
@@
 		(dnp no)
 		(fields_autoplaced yes)
-		(property "Reference" "J7"
+		(property "Reference" "J8"
 			(at 175.26 76.2 0)
 			(show_name no)
@@
 			)
 		)
-		(property "Footprint" "HDRV2W64P0X254_1X2_508X254X588P"
+		(property "Footprint" "SamacSys_Parts:HDRV2W64P0X254_1X2_508X254X588P"
 			(at 168.91 -8.56 0)
 			(hide yes)
@@
 			(project "Ročníkový projekt S3E"
 				(path "/c4e08560-2444-47e9-8324-16df61887a86/fbd34285-b602-47a7-9c37-182089d835a8"
-					(reference "J7")
+					(reference "J8")
 					(unit 1)
 				)
@@
 		(dnp no)
 		(fields_autoplaced yes)
-		(property "Reference" "S1"
+		(property "Reference" "S4"
 			(at 107.95 76.2 0)
 			(show_name no)
@@
 			)
 		)
-		(property "Footprint" "TACT67NF"
+		(property "Footprint" "My parts:TACT67NF"
 			(at 114.3 178.74 0)
 			(hide yes)
@@
 			(project "Ročníkový projekt S3E"
 				(path "/c4e08560-2444-47e9-8324-16df61887a86/fbd34285-b602-47a7-9c37-182089d835a8"
-					(reference "S1")
+					(reference "S4")
 					(unit 1)
 				)

Commit message: Auto-backup: 18:09:10 17/04/2026
Parts:
- renumbered J8 to J10, J6 to J8, J7 to J9
Connections:
- no-connect marks 0 -> 6
Changed lines of the file:
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@@
 	(generator_version "10.0")
 	(paper "A4")
+	(no_connect
+		(at 214.63 83.82)
+	)
+	(no_connect
+		(at 166.37 83.82)
+	)
+	(no_connect
+		(at 166.37 86.36)
+	)
+	(no_connect
+		(at 214.63 86.36)
+	)
+	(no_connect
+		(at 118.11 83.82)
+	)
+	(no_connect
+		(at 118.11 86.36)
+	)
 	(wire
 		(pts
@@
 			(width 0)
 			(type default)
-		)
-	)
-	(label ""
-		(at 30.48 82.55 0)
-		(effects
-			(font
-				(size 1.27 1.27)
-			)
-			(justify left bottom)
 		)
 	)
@@
 		(dnp no)
 		(fields_autoplaced yes)
-		(property "Reference" "J6"
+		(property "Reference" "J8"
 			(at 78.74 76.2 0)
 			(show_name no)
@@
 			(project "Ročníkový projekt S3E"
 				(path "/c4e08560-2444-47e9-8324-16df61887a86/fbd34285-b602-47a7-9c37-182089d835a8"
-					(reference "J6")
+					(reference "J8")
 					(unit 1)
 				)
@@
 		(dnp no)
 		(fields_autoplaced yes)
-		(property "Reference" "J7"
+		(property "Reference" "J9"
 			(at 127 76.2 0)
 			(show_name no)
@@
 			(project "Ročníkový projekt S3E"
 				(path "/c4e08560-2444-47e9-8324-16df61887a86/fbd34285-b602-47a7-9c37-182089d835a8"
-					(reference "J7")
+					(reference "J9")
 					(unit 1)
 				)
@@
 		(dnp no)
 		(fields_autoplaced yes)
-		(property "Reference" "J8"
+		(property "Reference" "J10"
 			(at 175.26 76.2 0)
 			(show_name no)
@@
 			(project "Ročníkový projekt S3E"
 				(path "/c4e08560-2444-47e9-8324-16df61887a86/fbd34285-b602-47a7-9c37-182089d835a8"
-					(reference "J8")
+					(reference "J10")
 					(unit 1)
 				)
