File: Display_Board.kicad_sch (KiCad schematic)
At the start: 2 parts

Commit message: Auto-backup: 09:05:42 15/04/2026
Parts:
- Conn2: value ~ -> (none)
Changed lines of the file:
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@@
 (kicad_sch
-	(version 20250114)
+	(version 20260306)
 	(generator "eeschema")
-	(generator_version "9.0")
+	(generator_version "10.0")
 	(paper "A4")
 	(junction
@@
 	)
 	(junction
-		(at 156.21 101.6)
-		(diameter 0)
-		(color 0 0 0 0)
-	)
-	(junction
 		(at 87.63 86.36)
 		(diameter 0)
@@
 		(property "Intersheetrefs" "${INTERSHEET_REFS}"
 			(at 133.13 76.2 0)
+			(hide yes)
+			(show_name no)
+			(do_not_autoplace no)
 			(effects
 				(font
@@
 				)
 				(justify left)
-				(hide yes)
 			)
 		)
@@
 		(property "Intersheetrefs" "${INTERSHEET_REFS}"
 			(at 133.13 81.28 0)
+			(hide yes)
+			(show_name no)
+			(do_not_autoplace no)
 			(effects
 				(font
@@
 				)
 				(justify left)
-				(hide yes)
 			)
 		)
@@
 		(property "Intersheetrefs" "${INTERSHEET_REFS}"
 			(at 58.7005 76.2 0)
+			(hide yes)
+			(show_name no)
+			(do_not_autoplace no)
 			(effects
 				(font
@@
 				)
 				(justify right)
-				(hide yes)
 			)
 		)
@@
 		(property "Intersheetrefs" "${INTERSHEET_REFS}"
 			(at 133.13 88.9 0)
+			(hide yes)
+			(show_name no)
+			(do_not_autoplace no)
 			(effects
 				(font
@@
 				)
 				(justify left)
-				(hide yes)
 			)
 		)
@@
 		(property "Intersheetrefs" "${INTERSHEET_REFS}"
 			(at 132.9486 78.74 0)
+			(hide yes)
+			(show_name no)
+			(do_not_autoplace no)
 			(effects
 				(font
@@
 				)
 				(justify left)
-				(hide yes)
 			)
 		)
@@
 		(property "Intersheetrefs" "${INTERSHEET_REFS}"
 			(at 58.7005 81.28 0)
+			(hide yes)
+			(show_name no)
+			(do_not_autoplace no)
 			(effects
 				(font
@@
 				)
 				(justify right)
-				(hide yes)
 			)
 		)
@@
 		(property "Intersheetrefs" "${INTERSHEET_REFS}"
 			(at 58.7005 73.66 0)
+			(hide yes)
+			(show_name no)
+			(do_not_autoplace no)
 			(effects
 				(font
@@
 				)
 				(justify right)
-				(hide yes)
 			)
 		)
@@
 		(property "Intersheetrefs" "${INTERSHEET_REFS}"
 			(at 133.13 73.66 0)
+			(hide yes)
+			(show_name no)
+			(do_not_autoplace no)
 			(effects
 				(font
@@
 				)
 				(justify left)
-				(hide yes)
 			)
 		)
@@
 		(property "Intersheetrefs" "${INTERSHEET_REFS}"
 			(at 62.45 88.9 0)
+			(hide yes)
+			(show_name no)
+			(do_not_autoplace no)
 			(effects
 				(font
@@
 				)
 				(justify right)
-				(hide yes)
 			)
 		)
@@
 		(property "Intersheetrefs" "${INTERSHEET_REFS}"
 			(at 132.9486 86.36 0)
+			(hide yes)
+			(show_name no)
+			(do_not_autoplace no)
 			(effects
 				(font
@@
 				)
 				(justify left)
-				(hide yes)
 			)
 		)
@@
 		(property "Intersheetrefs" "${INTERSHEET_REFS}"
 			(at 58.7005 86.36 0)
+			(hide yes)
+			(show_name no)
+			(do_not_autoplace no)
 			(effects
 				(font
@@
 				)
 				(justify right)
-				(hide yes)
 			)
 		)
@@
 		(property "Intersheetrefs" "${INTERSHEET_REFS}"
 			(at 58.7005 83.82 0)
+			(hide yes)
+			(show_name no)
+			(do_not_autoplace no)
 			(effects
 				(font
@@
 				)
 				(justify right)
-				(hide yes)
 			)
 		)
@@
 		(property "Intersheetrefs" "${INTERSHEET_REFS}"
 			(at 58.7005 78.74 0)
+			(hide yes)
+			(show_name no)
+			(do_not_autoplace no)
 			(effects
 				(font
@@
 				)
 				(justify right)
-				(hide yes)
 			)
 		)
@@
 		(property "Intersheetrefs" "${INTERSHEET_REFS}"
 			(at 133.009 83.82 0)
+			(hide yes)
+			(show_name no)
+			(do_not_autoplace no)
 			(effects
 				(font
@@
 				)
 				(justify left)
-				(hide yes)
 			)
 		)
@@
 		(at 97.79 71.12 0)
 		(unit 1)
+		(body_style 1)
 		(exclude_from_sim no)
 		(in_bom yes)
 		(on_board yes)
+		(in_pos_files yes)
 		(dnp no)
 		(fields_autoplaced yes)
 		(property "Reference" "Conn2"
 			(at 97.79 68.58 0)
+			(show_name no)
+			(do_not_autoplace no)
 			(effects
 				(font
@@
 			)
 		)
-		(property "Value" "~"
+		(property "Value" ""
 			(at 97.79 71.12 0)
+			(hide yes)
+			(show_name no)
+			(do_not_autoplace no)
 			(effects
 				(font
 					(size 1.27 1.27)
 				)
-				(hide yes)
 			)
 		)
 		(property "Footprint" "My parts:DIP-14_IDC_2x14"
 			(at 97.79 71.12 0)
+			(hide yes)
+			(show_name no)
+			(do_not_autoplace no)
 			(effects
 				(font
 					(size 1.27 1.27)
 				)
-				(hide yes)
 			)
 		)
 		(property "Datasheet" ""
 			(at 97.79 71.12 0)
+			(hide yes)
+			(show_name no)
+			(do_not_autoplace no)
 			(effects
 				(font
 					(size 1.27 1.27)
 				)
-				(hide yes)
 			)
 		)
 		(property "Description" ""
 			(at 97.79 71.12 0)
+			(hide yes)
+			(show_name no)
+			(do_not_autoplace no)
 			(effects
 				(font
 					(size 1.27 1.27)
 				)
-				(hide yes)
 			)
 		)
@@
 		)
 		(instances
-			(project ""
+			(project "Ročníkový projekt S3E"
 				(path "/c4e08560-2444-47e9-8324-16df61887a86/93b983ec-69c3-459b-8769-40a6a6507421"
 					(reference "Conn2")
@@
 		(at 179.07 73.66 0)
 		(unit 1)
+		(body_style 1)
 		(exclude_from_sim no)
 		(in_bom yes)
 		(on_board yes)
+		(in_pos_files yes)
 		(dnp no)
 		(fields_autoplaced yes)
 		(property "Reference" "S1"
 			(at 190.7249 66.04 0)
+			(show_name no)
+			(do_not_autoplace no)
 			(effects
 				(font
@@
 		(property "Value" "S"
 			(at 187.706 66.548 0)
+			(hide yes)
+			(show_name no)
+			(do_not_autoplace no)
 			(effects
 				(font
@@
 				)
 				(justify left top)
-				(hide yes)
 			)
 		)
 		(property "Footprint" "My parts:Patice_display"
 			(at 198.12 168.58 0)
+			(hide yes)
+			(show_name no)
+			(do_not_autoplace no)
 			(effects
 				(font
@@
 				)
 				(justify left top)
-				(hide yes)
 			)
 		)
 		(property "Datasheet" ""
 			(at 198.12 268.58 0)
+			(hide yes)
+			(show_name no)
+			(do_not_autoplace no)
 			(effects
 				(font
@@
 				)
 				(justify left top)
-				(hide yes)
 			)
 		)
 		(property "Description" ""
 			(at 174.752 62.992 0)
+			(hide yes)
+			(show_name no)
+			(do_not_autoplace no)
 			(effects
 				(font
 					(size 1.27 1.27)
 				)
-				(hide yes)
 			)
 		)
@@
 		)
 		(instances
-			(project ""
+			(project "Ročníkový projekt S3E"
 				(path "/c4e08560-2444-47e9-8324-16df61887a86/93b983ec-69c3-459b-8769-40a6a6507421"
 					(reference "S1")

Commit message: Auto-backup: 10:53:27 17/04/2026
Parts:
- removed S1: S, My parts:Patice_display, symbol My_parts:Screen_connector_symbol
- added S1, S2: (no value), My parts:DIP 18 Patice Display Digit 1, symbol My_parts:Digit_1
- added S3: (no value), My parts:DIP-10 Patice Display Digit 3 4, symbol My_parts:Digit_3_4
Connections:
- net A' renamed B
- net B: now also S1.10 (B), S1.15 (B), S2.10 (B), S2.15 (B), S3.9 (B)
- net B' renamed A
- net A: now also S1.11 (A), S1.16 (A), S2.11 (A), S2.16 (A), S3.3 (A)
- net C' renamed DP
- net DP: now also S1.4 (DP), S1.9 (DP), S2.4 (DP), S2.9 (DP), S3.2 (DP)
- net D' renamed C
- net C: now also S1.3 (C), S1.8 (C), S2.3 (C), S2.8 (C), S3.8 (C)
- net DIGIT_1 renamed D1
- net D1: now also S3.5 (Anode2)
- net DIGIT_2 renamed D2
- net D2: now also S3.10 (Anode1)
- net DIGIT_3 renamed D3
- net D3: now also S2.14 (Anode1)
- net DIGIT_4 renamed D4
- net D4: now also S2.13 (Anode2)
- net DIGIT_5 renamed D5
- net D5: now also S1.14 (Anode1)
- net DIGIT_6 renamed D6
- net D6: now also S1.13 (Anode2)
- net DP' renamed G
- net G: now also S1.17 (G), S1.7 (G), S2.17 (G), S2.7 (G), S3.1 (G)
- net E' renamed D
- net D: now also S1.2 (D), S1.6 (D), S2.2 (D), S2.6 (D), S3.6 (D)
- net F' renamed E
- net E: now also S1.1 (E), S1.5 (E), S2.1 (E), S2.5 (E), S3.7 (E)
- net G' renamed F
- net F: now also S1.12 (F), S1.18 (F), S2.12 (F), S2.18 (F), S3.4 (F)

Commit message: Auto-backup: 18:09:10 17/04/2026
Parts:
- renumbered Conn2 to J7
